File: hardware/eagle/rev_a/button.sch (EAGLE design)
At the start: 13 parts

Commit message: First stab at button board Fits current body model, faceplate needs spacing of start/select
Parts:
- added JP2: (no value), SparkFun-Connectors:M04PTH
- added PWRON: SKPDAMD010, switches:SKPDAMD010
- SELECT, START: value SKPDAMD010 -> EVQ11D09K; device switches:SKPDAMD010 -> BMO:EVQ11D09K
- renumbered U$1 to TEENSY
Connections:
- new net N$2: JP2.4, PWRON.P$2
- new net PROGRAM: JP2.3, TEENSY.PROGRAM
- new net VCC: JP2.1, TEENSY.VIN
- net GND: now also JP2.2, PWRON.P$1; no longer TEENSY.GND2
- net N$14: now also RB.2
