File: hardware/eagle/rev_a/usb.sch (EAGLE design)
At the start: 41 parts, among them J1 MICRO_USB_B_HIROSE_ZX62-B-5PA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, P1 1932638-3_TE_AMP, P2 1932638-3_TE_AMP, P3 USB-A-FEMALETESTPOINT, U1 TPS2043B, U2 SN75240, U3 SN75240, U4 SN75240, U5 TUSB2036VF, X1 ABMM-6.000MHZ-B2-T

Commit message: Added boards for back buttons and charging/serial port Tweaks and redesigns for button/usb boards to fit in case better
Parts:
- P1, P2: value 1932638-3_TE_AMP -> USB-A-FEMALE; device BMO:1932638-3_TE_AMP -> BMO:USB-A-FEMALE
Changed lines of the file:
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@@
 <part name="U5" library="BMO" deviceset="TUSB2036VF" device=""/>
 <part name="U1" library="BMO" deviceset="TPS2043B" device=""/>
-<part name="P1" library="BMO" deviceset="1932638-3_TE_AMP" device=""/>
-<part name="P2" library="BMO" deviceset="1932638-3_TE_AMP" device=""/>
 <part name="GND2" library="umich" deviceset="GND" device=""/>
 <part name="GND1" library="umich" deviceset="GND" device=""/>
@@
 <part name="JP1" library="SparkFun-Connectors" deviceset="M03" device="PTH"/>
 <part name="C15" library="passives" deviceset="CAPACITOR" device="" value="0.1u"/>
+<part name="P1" library="BMO" deviceset="USB-A-FEMALE" device=""/>
+<part name="P2" library="BMO" deviceset="USB-A-FEMALE" device=""/>
 </parts>
 <sheets>
@@
 <instance part="U5" gate="A" x="45.72" y="111.76"/>
 <instance part="U1" gate="G$1" x="142.24" y="50.8"/>
-<instance part="P1" gate="G$1" x="228.6" y="86.36"/>
-<instance part="P2" gate="G$1" x="228.6" y="124.46"/>
 <instance part="GND2" gate="1" x="76.2" y="68.58"/>
 <instance part="GND1" gate="1" x="15.24" y="68.58"/>
@@
 <instance part="JP1" gate="G$1" x="190.5" y="43.18"/>
 <instance part="C15" gate="G$1" x="7.62" y="96.52"/>
+<instance part="P1" gate="G$1" x="228.6" y="86.36"/>
+<instance part="P2" gate="G$1" x="228.6" y="124.46"/>
 </instances>
 <busses>
@@
 </segment>
 <segment>
-<pinref part="P2" gate="G$1" pin="GND"/>
-<wire x1="223.52" y1="121.92" x2="220.98" y2="121.92" width="0.1524" layer="91"/>
 <wire x1="220.98" y1="121.92" x2="220.98" y2="106.68" width="0.1524" layer="91"/>
 <wire x1="220.98" y1="106.68" x2="218.44" y2="106.68" width="0.1524" layer="91"/>
@@
 <pinref part="GND8" gate="1" pin="GND"/>
 <junction x="218.44" y="106.68"/>
+<pinref part="P2" gate="G$1" pin="GND"/>
+<wire x1="223.52" y1="121.92" x2="220.98" y2="121.92" width="0.1524" layer="91"/>
 </segment>
 <segment>
@@
 <junction x="218.44" y="71.12"/>
 <pinref part="P1" gate="G$1" pin="GND"/>
-<wire x1="223.52" y1="83.82" x2="220.98" y2="83.82" width="0.1524" layer="91"/>
+<wire x1="220.98" y1="83.82" x2="223.52" y2="83.82" width="0.1524" layer="91"/>
 </segment>
 <segment>
@@
 <junction x="167.64" y="119.38"/>
 <pinref part="P1" gate="G$1" pin="D-"/>
-<wire x1="187.96" y1="88.9" x2="223.52" y2="88.9" width="0.1524" layer="91"/>
+<wire x1="223.52" y1="88.9" x2="187.96" y2="88.9" width="0.1524" layer="91"/>
 </segment>
 </net>
@@
 <junction x="185.42" y="109.22"/>
 <pinref part="P1" gate="G$1" pin="D+"/>
-<wire x1="185.42" y1="86.36" x2="223.52" y2="86.36" width="0.1524" layer="91"/>
+<wire x1="223.52" y1="86.36" x2="185.42" y2="86.36" width="0.1524" layer="91"/>
 </segment>
 </net>
@@
 <segment>
 <wire x1="190.5" y1="147.32" x2="190.5" y2="124.46" width="0.1524" layer="91"/>
+<pinref part="R4" gate="G$1" pin="2"/>
+<wire x1="187.96" y1="147.32" x2="190.5" y2="147.32" width="0.1524" layer="91"/>
 <pinref part="P2" gate="G$1" pin="D+"/>
 <wire x1="223.52" y1="124.46" x2="190.5" y2="124.46" width="0.1524" layer="91"/>
-<pinref part="R4" gate="G$1" pin="2"/>
-<wire x1="187.96" y1="147.32" x2="190.5" y2="147.32" width="0.1524" layer="91"/>
 </segment>
 </net>
 <net name="N$10" class="0">
 <segment>
-<pinref part="P2" gate="G$1" pin="D-"/>
-<wire x1="223.52" y1="127" x2="193.04" y2="127" width="0.1524" layer="91"/>
 <wire x1="193.04" y1="127" x2="193.04" y2="154.94" width="0.1524" layer="91"/>
 <pinref part="R3" gate="G$1" pin="2"/>
 <wire x1="193.04" y1="154.94" x2="187.96" y2="154.94" width="0.1524" layer="91"/>
+<pinref part="P2" gate="G$1" pin="D-"/>
+<wire x1="223.52" y1="127" x2="193.04" y2="127" width="0.1524" layer="91"/>
 </segment>
 </net>
@@
 <wire x1="215.9" y1="81.28" x2="215.9" y2="91.44" width="0.1524" layer="91"/>
 <pinref part="P1" gate="G$1" pin="+5V"/>
-<wire x1="215.9" y1="91.44" x2="223.52" y2="91.44" width="0.1524" layer="91"/>
+<wire x1="223.52" y1="91.44" x2="215.9" y2="91.44" width="0.1524" layer="91"/>
 <junction x="215.9" y="91.44"/>
 </segment>
@@
 <net name="N$4" class="0">
 <segment>
-<pinref part="P2" gate="G$1" pin="+5V"/>
-<wire x1="223.52" y1="129.54" x2="215.9" y2="129.54" width="0.1524" layer="91"/>
 <wire x1="215.9" y1="129.54" x2="203.2" y2="129.54" width="0.1524" layer="91"/>
 <wire x1="203.2" y1="129.54" x2="203.2" y2="76.2" width="0.1524" layer="91"/>
@@
 <pinref part="C10" gate="G$1" pin="1"/>
 <wire x1="215.9" y1="116.84" x2="215.9" y2="129.54" width="0.1524" layer="91"/>
+<pinref part="P2" gate="G$1" pin="+5V"/>
+<wire x1="223.52" y1="129.54" x2="215.9" y2="129.54" width="0.1524" layer="91"/>
 <junction x="215.9" y="129.54"/>
 </segment>
