File: hardware/bmo_power/charge_reg.kicad_sch (KiCad schematic)
At the start: 50 parts, among them U1 BQ25606RGET, U4 TPS61088RHLR, U5 LTC4412xS6, U6 SIA445EDJ-T1-GE3, U7 SIA445EDJ-T1-GE3

Commit message: embed 3d models
Connections:
- net BOOST_OUT: no longer U7.2, U7.5, U7.6
- net VBUS: no longer U6.2, U6.5, U6.6
